File: attiny84_bo.brd (EAGLE design)
At the start: 36 x 20 mm, 9 parts, among them J1 AVR_SPI_PRG_6NS, Y1 16MHz

Commit message: initial placement
Parts:
- moved LED1 16.2 mm to (18.8, 17.7), turned to 90 degrees
- moved J1 3.83 mm to (12.1, 13.3)
- moved C1 3.59 mm to (26.8, 13.1)
- moved U$1 3.59 mm to (20.4, 13.2)
- moved CX0 3.59 mm to (16.0, 13.1)
- moved CX1 3.59 mm to (24.1, 13.2)
- moved Y1 3.59 mm to (20.1, 13.2)
- moved C2 0.13 mm to (29.6, 5.46), turned to 90 degrees
Connections:
- new net N$6: JP1.10, U$1.5
- net +5V: now also JP1.2, LED1.A
- net GND: now also JP1.16, JP1.4, JP1.6, JP1.8
- net N$1: now also LED1.C
- net PB0/XTAL1: now also JP1.14
- net PB1/XTAL2: now also JP1.12
Changed lines of the file:
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@@
 <text x="8.255" y="1.016" size="1.016" layer="25" font="vector">http://helsinki.hacklab.fi</text>
 <text x="7.874" y="18.542" size="1.016" layer="25" font="vector">ATT84iny breakout board</text>
-<text x="4.064" y="12.827" size="1.016" layer="25" font="vector" rot="R270">ISP</text>
+<text x="8.001" y="12.319" size="1.016" layer="25" font="vector" rot="R270">ISP</text>
 </plain>
 <attributes>
@@
 <param name="mdDrill" value="10mil"/>
 <param name="mdSmdStop" value="0mil"/>
-<param name="msWidth" value="8mil"/>
+<param name="msWidth" value="6mil"/>
 <param name="msDrill" value="12mil"/>
 <param name="msMicroVia" value="12mil"/>
@@
 </autorouter>
 <elements>
-<element name="J1" library="SparkFun-Connectors" package="2X3-NS" value="AVR_SPI_PRG_6NS" x="8.255" y="13.716" smashed="yes" rot="R90"/>
-<element name="C1" library="rcl" package="C0805" value="" x="23.241" y="13.589" smashed="yes" rot="R270">
-<attribute name="VALUE" x="20.701" y="14.859" size="1.27" layer="27" rot="R270"/>
+<element name="J1" library="SparkFun-Connectors" package="2X3-NS" value="AVR_SPI_PRG_6NS" x="12.065" y="13.335" smashed="yes" rot="R90"/>
+<element name="C1" library="rcl" package="C0805" value="" x="26.797" y="13.081" smashed="yes" rot="R270">
+<attribute name="VALUE" x="24.257" y="14.351" size="1.27" layer="27" rot="R270"/>
 </element>
-<element name="LED1" library="SparkFun-LED" package="LED-0603" value="" x="2.667" y="18.796" smashed="yes" rot="R270">
-<attribute name="VALUE" x="1.651" y="17.7165" size="0.4064" layer="27"/>
+<element name="LED1" library="SparkFun-LED" package="LED-0603" value="" x="18.796" y="17.653" smashed="yes" rot="R90">
+<attribute name="VALUE" x="19.812" y="18.7325" size="0.4064" layer="27" rot="R180"/>
 </element>
-<element name="C2" library="rcl" package="C0805" value="" x="29.591" y="5.588" smashed="yes" rot="R270">
-<attribute name="VALUE" x="27.051" y="6.858" size="1.27" layer="27" rot="R270"/>
+<element name="C2" library="rcl" package="C0805" value="" x="29.591" y="5.461" smashed="yes" rot="R90">
+<attribute name="VALUE" x="32.131" y="4.191" size="1.27" layer="27" rot="R90"/>
 </element>
-<element name="CX0" library="rcl" package="C0603" value="22pF" x="12.446" y="13.589" smashed="yes" rot="MR90"/>
-<element name="CX1" library="rcl" package="C0603" value="22pF" x="20.574" y="13.716" smashed="yes" rot="MR270"/>
-<element name="Y1" library="SparkFun-FreqCtrl" package="CRYSTAL-SMD-5X3" value="16MHz" x="16.51" y="13.716" smashed="yes" rot="MR0"/>
-<element name="U$1" library="SparkFun-DigitalIC" package="SO14" value="ATTINY84" x="16.891" y="13.716" rot="R180"/>
+<element name="CX0" library="rcl" package="C0603" value="22pF" x="16.002" y="13.081" smashed="yes" rot="MR90"/>
+<element name="CX1" library="rcl" package="C0603" value="22pF" x="24.13" y="13.208" smashed="yes" rot="MR270"/>
+<element name="Y1" library="SparkFun-FreqCtrl" package="CRYSTAL-SMD-5X3" value="16MHz" x="20.066" y="13.208" smashed="yes" rot="MR0"/>
+<element name="U$1" library="SparkFun-DigitalIC" package="SO14" value="ATTINY84" x="20.447" y="13.208" rot="R180"/>
 <element name="JP1" library="pinhead" package="2X08" value="" x="17.653" y="5.588" smashed="yes" rot="R180">
 <attribute name="VALUE" x="27.813" y="10.033" size="1.27" layer="27" rot="R180"/>
@@
 <contactref element="C2" pad="2"/>
 <contactref element="U$1" pad="14"/>
+<contactref element="JP1" pad="16"/>
+<contactref element="JP1" pad="4"/>
+<contactref element="JP1" pad="8"/>
+<contactref element="JP1" pad="6"/>
 </signal>
 <signal name="+5V" class="1">
@@
 <contactref element="C2" pad="1"/>
 <contactref element="U$1" pad="1"/>
-<wire x1="20.701" y1="16.516" x2="23.241" y2="14.539" width="0" layer="19" extent="1-1"/>
-<wire x1="29.591" y1="6.538" x2="23.241" y2="14.539" width="0" layer="19" extent="1-1"/>
-<wire x1="6.985" y1="11.176" x2="20.701" y2="16.516" width="0" layer="19" extent="1-1"/>
+<contactref element="JP1" pad="2"/>
+<contactref element="LED1" pad="A"/>
+<wire x1="24.257" y1="16.008" x2="26.797" y2="14.031" width="0" layer="19" extent="1-1"/>
+<wire x1="19.546" y1="17.653" x2="24.257" y2="16.008" width="0" layer="19" extent="1-1"/>
+<wire x1="26.543" y1="4.318" x2="26.797" y2="14.031" width="0" layer="19" extent="1-1"/>
+<wire x1="29.591" y1="4.511" x2="26.543" y2="4.318" width="0" layer="19" extent="1-1"/>
+<wire x1="10.795" y1="10.795" x2="19.546" y2="17.653" width="0" layer="19" extent="1-1"/>
 </signal>
 <signal name="PB0/XTAL1">
@@
 <contactref element="Y1" pad="1"/>
 <contactref element="U$1" pad="2"/>
-<wire x1="18.36" y1="12.566" x2="20.574" y2="12.866" width="0" layer="19" extent="16-16"/>
-<wire x1="19.431" y1="16.516" x2="20.574" y2="12.866" width="0" layer="19" extent="1-16"/>
+<contactref element="JP1" pad="14"/>
+<wire x1="24.13" y1="12.358" x2="22.987" y2="16.008" width="0" layer="19" extent="1-16"/>
+<wire x1="21.916" y1="12.058" x2="24.13" y2="12.358" width="0" layer="19" extent="16-16"/>
+<wire x1="11.303" y1="4.318" x2="21.916" y2="12.058" width="0" layer="19" extent="16-16"/>
 </signal>
 <signal name="PB1/XTAL2">
@@
 <contactref element="Y1" pad="3"/>
 <contactref element="U$1" pad="3"/>
-<wire x1="14.66" y1="14.866" x2="18.161" y2="16.516" width="0" layer="19" extent="1-16"/>
-<wire x1="12.446" y1="14.439" x2="14.66" y2="14.866" width="0" layer="19" extent="16-16"/>
+<contactref element="JP1" pad="12"/>
+<wire x1="18.216" y1="14.358" x2="21.717" y2="16.008" width="0" layer="19" extent="1-16"/>
+<wire x1="16.002" y1="13.931" x2="18.216" y2="14.358" width="0" layer="19" extent="16-16"/>
+<wire x1="13.843" y1="4.318" x2="16.002" y2="13.931" width="0" layer="19" extent="16-16"/>
 </signal>
 <signal name="PB3/RESET-">
 <contactref element="U$1" pad="4"/>
 <contactref element="J1" pad="5"/>
-<wire x1="9.525" y1="16.256" x2="16.891" y2="16.516" width="0" layer="19" extent="1-1"/>
+<wire x1="13.335" y1="15.875" x2="20.447" y2="16.008" width="0" layer="19" extent="1-1"/>
 </signal>
 <signal name="PA6/MOSI">
@@
 <contactref element="U$1" pad="7"/>
 <contactref element="JP1" pad="13"/>
-<wire x1="6.985" y1="13.716" x2="13.081" y2="16.516" width="0" layer="19" extent="1-1"/>
-<wire x1="11.303" y1="6.858" x2="6.985" y2="13.716" width="0" layer="19" extent="1-1"/>
+<wire x1="10.795" y1="13.335" x2="16.637" y2="16.008" width="0" layer="19" extent="1-1"/>
+<wire x1="11.303" y1="6.858" x2="10.795" y2="13.335" width="0" layer="19" extent="1-1"/>
 </signal>
 <signal name="PA5/MISO">
@@
 <contactref element="U$1" pad="8"/>
 <contactref element="JP1" pad="11"/>
-<wire x1="9.525" y1="11.176" x2="13.081" y2="10.916" width="0" layer="19" extent="1-1"/>
-<wire x1="13.843" y1="6.858" x2="13.081" y2="10.916" width="0" layer="19" extent="1-1"/>
+<wire x1="13.335" y1="10.795" x2="16.637" y2="10.408" width="0" layer="19" extent="1-1"/>
+<wire x1="13.843" y1="6.858" x2="13.335" y2="10.795" width="0" layer="19" extent="1-1"/>
 </signal>
 <signal name="PA4/SCL">
@@
 <contactref element="U$1" pad="9"/>
 <contactref element="JP1" pad="9"/>
-<wire x1="16.383" y1="6.858" x2="14.351" y2="10.916" width="0" layer="19" extent="1-1"/>
-<wire x1="9.525" y1="13.716" x2="14.351" y2="10.916" width="0" layer="19" extent="1-1"/>
+<wire x1="16.383" y1="6.858" x2="17.907" y2="10.408" width="0" layer="19" extent="1-1"/>
+<wire x1="13.335" y1="13.335" x2="17.907" y2="10.408" width="0" layer="19" extent="1-1"/>
 </signal>
 <signal name="N$1">
 <contactref element="U$1" pad="6"/>
 <contactref element="JP1" pad="15"/>
-<wire x1="8.763" y1="6.858" x2="14.351" y2="16.516" width="0" layer="19" extent="1-1"/>
+<contactref element="LED1" pad="C"/>
+<wire x1="18.046" y1="17.653" x2="17.907" y2="16.008" width="0" layer="19" extent="1-1"/>
+<wire x1="8.763" y1="6.858" x2="17.907" y2="16.008" width="0" layer="19" extent="1-1"/>
 </signal>
 <signal name="N$2">
 <contactref element="U$1" pad="10"/>
 <contactref element="JP1" pad="7"/>
-<wire x1="18.923" y1="6.858" x2="15.621" y2="10.916" width="0" layer="19" extent="1-1"/>
+<wire x1="18.923" y1="6.858" x2="19.177" y2="10.408" width="0" layer="19" extent="1-1"/>
 </signal>
 <signal name="N$3">
 <contactref element="U$1" pad="11"/>
 <contactref element="JP1" pad="5"/>
-<wire x1="21.463" y1="6.858" x2="16.891" y2="10.916" width="0" layer="19" extent="1-1"/>
+<wire x1="21.463" y1="6.858" x2="20.447" y2="10.408" width="0" layer="19" extent="1-1"/>
 </signal>
 <signal name="N$4">
 <contactref element="U$1" pad="12"/>
 <contactref element="JP1" pad="3"/>
-<wire x1="24.003" y1="6.858" x2="18.161" y2="10.916" width="0" layer="19" extent="1-1"/>
+<wire x1="24.003" y1="6.858" x2="21.717" y2="10.408" width="0" layer="19" extent="1-1"/>
 </signal>
 <signal name="N$5">
 <contactref element="U$1" pad="13"/>
 <contactref element="JP1" pad="1"/>
-<wire x1="19.431" y1="10.916" x2="26.543" y2="6.858" width="0" layer="19" extent="1-1"/>
+<wire x1="26.543" y1="6.858" x2="22.987" y2="10.408" width="0" layer="19" extent="1-1"/>
+</signal>
+<signal name="N$6">
+<contactref element="U$1" pad="5"/>
+<contactref element="JP1" pad="10"/>
+<wire x1="16.383" y1="4.318" x2="19.177" y2="16.008" width="0" layer="19" extent="1-1"/>
 </signal>
 </signals>
