File: attiny4313_bo.brd (EAGLE design)
At the start: 49.5 x 22.2 mm, 11 parts, among them J1 AVR_SPI_PRG_6NS, Y1 16MHz

Commit message: signals v1, probably bad
Parts:
- moved C1 9.96 mm to (32.4, 11.4), turned to 90 degrees
- moved J1 5.47 mm to (38.7, 17.1), turned to 180 degrees
- moved U$1 2.41 mm to (24.1, 14.4)
- moved CX0 2.22 mm to (19.4, 14.0)
- moved CX1 2.22 mm to (27.4, 14.1)
- moved Y1 2.22 mm to (23.5, 14.1)
- moved C2 1.40 mm to (8.89, 3.81), turned to 90 degrees
- moved H1 1.17 mm to (4.95, 11.0)
- moved H2 1.09 mm to (45.5, 10.8)
- moved JP1 0.57 mm to (23.4, 4.19), turned to 180 degrees
Connections:
- removed net N$1: CX0.2, U$1.5, Y1.3
- removed net N$2: LED1.C
- removed net PB0/XTAL1: CX1.2, U$1.4, Y1.1
- new net PA0/XTAL1: CX0.2, JP1.19, U$1.5, Y1.3
- new net PA1/XTAL2: CX1.2, JP1.17, U$1.4, Y1.1
- new net PD0/RDX: JP1.16, U$1.2
- new net PD1/TXD: JP1.14, U$1.3
- new net PD2: JP1.12, U$1.6
- new net PD3: JP1.10, U$1.7
- new net PD4: JP1.8, U$1.8
- new net PD5: JP1.6, U$1.9
- new net PD6: JP1.4, LED1.C, U$1.11
- net +5V: now also JP1.18
- net PB0: now also JP1.15; no longer JP1.1
- net PB1: now also JP1.13; no longer JP1.3
- net PB2: now also JP1.11; no longer JP1.5
- net PB3: now also JP1.9; no longer JP1.7
- net PB4: now also JP1.7; no longer JP1.9
- net PB5/MOSI: now also JP1.5; no longer JP1.13
- net PB6/MISO: now also JP1.3; no longer JP1.11
- net PB7/SCL: now also JP1.1; no longer JP1.15

Commit message: pin identifiers
Parts:
- moved LED1 10.7 mm to (15.4, 10.7), turned to 270 degrees
- moved C2 1.82 mm to (10.5, 4.57)
- moved JP1 1.69 mm to (25.0, 4.57)
- moved J1 1.25 mm to (37.6, 16.6)
Connections:
- net +5V: now also JP1.20; no longer JP1.18
- net GND: now also JP1.18; no longer JP1.20
- net PD0/RDX: now also JP1.4; no longer JP1.16
- net PD1/TXD: now also JP1.6; no longer JP1.14
- net PD2: now also JP1.8; no longer JP1.12
- net PD4: now also JP1.12; no longer JP1.8
- net PD5: now also JP1.14; no longer JP1.6
- net PD6: now also JP1.16; no longer JP1.4
Other:
- board text added: "5V GND PD6 PD5 PD4 PD3 PD2 RX TX 5V"
- board text added: "5V RX TX PD2 PD3 PD4 PD5 PD6 GND 5V"
- board text added: "PA0 PA1 PB0 PB1 PB2 PB3 PB4 PB5 PB6 PB7"
- board text added: "PB7 PB6 PB5 PB4 PB3 PB2 PB1 PB0 PA1 PA0"
- board text removed: "5V GND GND GND PB2 PB1 PB0 5V"
- board text removed: "5V PB0 PB1 PB2 GND GND GND 5V"
- board text removed: "PA0 PA1 PA2 PA3 PA4 PA5 PA6 PA7"
- board text removed: "PA7 PA6 PA5 PA4 PA3 PA2 PA1 PA0"

Commit message: routed
Routing:
- net +5V: track 0.00 -> 52.6 mm
- net PD2: track 0.00 -> 49.2 mm
- net PB1: track 0.00 -> 39.1 mm, vias 0 -> 2
- net PB5/MOSI: track 0.00 -> 38.2 mm, vias 0 -> 1
- net PD4: track 0.00 -> 37.4 mm, vias 0 -> 1
- net PD3: track 0.00 -> 33.0 mm, vias 0 -> 2
- net PD1/TXD: track 0.00 -> 32.4 mm, vias 0 -> 1
- net PB6/MISO: track 0.00 -> 32.1 mm, vias 0 -> 2
- net PA1/XTAL2: track 0.00 -> 24.7 mm, vias 0 -> 2
- net PB7/SCL: track 0.00 -> 23.6 mm, vias 0 -> 1
- net PB3: track 0.00 -> 20.5 mm, vias 0 -> 2
- net PD5: track 0.00 -> 20.5 mm, vias 0 -> 1
- net PA0/XTAL1: track 0.00 -> 19.0 mm, vias 0 -> 1
- net PD0/RDX: track 0.00 -> 18.1 mm, vias 0 -> 2
- net PB4: track 0.00 -> 12.1 mm, vias 0 -> 1
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
Commit message: minor adjustments
Routing:
- net GND: vias 3 -> 12
Changed lines of the file:
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@@
 <setting verticaltext="up"/>
 </settings>
-<grid distance="5" unitdist="mil" unit="mil" style="lines" multiple="1" display="yes" altdistance="196.850394" altunitdist="mil" altunit="mil"/>
+<grid distance="5" unitdist="mil" unit="mm" style="lines" multiple="1" display="yes" altdistance="196.850394" altunitdist="mil" altunit="mil"/>
 <layers>
 <layer number="1" name="Top" color="4" fill="1" visible="yes" active="yes"/>
@@
 <wire x1="18.4912" y1="17.9832" x2="18.4634" y2="17.99941875" width="0.254" layer="1"/>
 <via x="18.288" y="15.748" extent="1-16" drill="0.3048"/>
+<via x="35.687" y="8.763" extent="1-16" drill="0.3048"/>
+<via x="36.957" y="7.874" extent="1-16" drill="0.3048"/>
+<via x="26.162" y="7.874" extent="1-16" drill="0.3048"/>
+<via x="32.512" y="18.796" extent="1-16" drill="0.3048"/>
+<via x="41.021" y="12.954" extent="1-16" drill="0.3048"/>
+<via x="39.624" y="6.604" extent="1-16" drill="0.3048"/>
+<via x="32.258" y="15.875" extent="1-16" drill="0.3048"/>
+<via x="14.986" y="18.669" extent="1-16" drill="0.3048"/>
+<via x="14.224" y="14.478" extent="1-16" drill="0.3048"/>
 </signal>
 <signal name="+5V" class="1">
@@
 <wire x1="20.4216" y1="9.3472" x2="22.5552" y2="9.3472" width="0.1524" layer="1"/>
 <wire x1="20.4216" y1="11.7856" x2="20.4216" y2="9.3472" width="0.1524" layer="1"/>
-<wire x1="19.5072" y1="12.7" x2="20.4216" y2="11.7856" width="0.1524" layer="1"/>
-<wire x1="18.3896" y1="12.7" x2="19.5072" y2="12.7" width="0.1524" layer="1"/>
-<wire x1="18.3896" y1="12.3952" x2="18.3896" y2="12.7" width="0.1524" layer="1"/>
+<wire x1="19.5072" y1="12.573" x2="20.4216" y2="11.7856" width="0.1524" layer="1"/>
+<wire x1="18.3896" y1="12.573" x2="19.5072" y2="12.573" width="0.1524" layer="1"/>
+<wire x1="18.3896" y1="12.3952" x2="18.3896" y2="12.573" width="0.1524" layer="1"/>
 <wire x1="18.288" y1="12.2936" x2="18.3896" y2="12.3952" width="0.1524" layer="16"/>
 <wire x1="18.288" y1="11.9888" x2="18.288" y2="12.2936" width="0.1524" layer="16"/>
@@
 <wire x1="40.9448" y1="16.256" x2="40.9448" y2="16.5608" width="0.1524" layer="1"/>
 <wire x1="41.8592" y1="15.3416" x2="40.9448" y2="16.256" width="0.1524" layer="1"/>
-<wire x1="41.8592" y1="11.684" x2="41.8592" y2="15.3416" width="0.1524" layer="1"/>
-<wire x1="38.3032" y1="8.128" x2="41.8592" y2="11.684" width="0.1524" layer="1"/>
-<wire x1="38.3032" y1="2.4384" x2="38.3032" y2="8.128" width="0.1524" layer="1"/>
-<wire x1="37.2872" y1="1.4224" x2="38.3032" y2="2.4384" width="0.1524" layer="1"/>
+<wire x1="41.8592" y1="12.192" x2="41.8592" y2="15.3416" width="0.1524" layer="1"/>
+<wire x1="41.0972" y1="11.049" x2="41.8592" y2="12.192" width="0.1524" layer="1"/>
+<wire x1="41.0972" y1="4.5974" x2="41.0972" y2="11.049" width="0.1524" layer="1"/>
+<wire x1="37.2872" y1="1.4224" x2="41.0972" y2="4.5974" width="0.1524" layer="1"/>
 <wire x1="28.8544" y1="1.4224" x2="37.2872" y2="1.4224" width="0.1524" layer="1"/>
 <wire x1="28.8544" y1="3.2512" x2="28.8544" y2="1.4224" width="0.1524" layer="1"/>
@@
 </signal>
 </signals>
+<errors>
+</errors>
 </board>
 </drawing>
