File: attiny4313_bo.brd (EAGLE design)
At the start: 49.5 x 22.2 mm, 11 parts, among them J1 AVR_SPI_PRG_6NS, Y1 16MHz

Commit message: minor adjustments
Routing:
- net GND: vias 12 -> 13
Other:
- board text added: "led optional"
- board text removed: "led (top) optional"
Changed lines of the file:
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@@
 <text x="12.319" y="7.874" size="0.7112" layer="25" font="vector">PA0 PA1 PB0 PB1 PB2 PB3 PB4 PB5 PB6 PB7</text>
 <text x="12.7" y="0.762" size="0.7112" layer="25" font="vector">5V  GND PD6 PD5 PD4 PD3 PD2 RX TX  5V</text>
-<text x="18.288" y="14.097" size="0.7112" layer="26" font="vector" rot="MR0">XTAL optional</text>
-<text x="18.288" y="12.446" size="0.7112" layer="26" font="vector" rot="MR0">led (top) optional</text>
+<text x="28.448" y="18.542" size="0.7112" layer="26" font="vector" rot="MR0">XTAL optional</text>
+<text x="12.954" y="16.129" size="0.7112" layer="25" font="vector" rot="R270">led optional</text>
 <text x="8.763" y="3.302" size="0.7112" layer="25" font="vector" rot="R90">10uF</text>
 <text x="34.29" y="10.16" size="0.7112" layer="25" font="vector" rot="R90">10uF</text>
-<text x="18.415" y="15.748" size="0.8128" layer="26" rot="MR0">12pF caps for xtal</text>
+<text x="29.845" y="17.145" size="0.7112" layer="26" rot="MR0">12pF caps for xtal</text>
 </plain>
 <attributes>
@@
 <via x="14.986" y="18.669" extent="1-16" drill="0.3048"/>
 <via x="14.224" y="14.478" extent="1-16" drill="0.3048"/>
+<via x="30.988" y="9.017" extent="1-16" drill="0.3048"/>
 </signal>
 <signal name="+5V" class="1">
