File: attiny1634_bo.brd (EAGLE design)
At the start: 49.5 x 22.2 mm, 11 parts, among them J1 AVR_SPI_PRG_6NS, Y1 12MHz

Commit message: adjusted texts and positions
Parts:
- moved C1 6.62 mm to (31.9, 18.0), turned to 270 degrees
- moved LED1 3.97 mm to (15.9, 14.6), turned to 0 degrees
- moved CX0 2.57 mm to (22.0, 13.6), turned to 270 degrees
- moved Y1 1.45 mm to (24.9, 14.5), turned to 270 degrees
- moved CX1 1.33 mm to (27.8, 15.4), turned to 90 degrees
- moved U$1 0.99 mm to (20.1, 14.6)
- moved J1 0.46 mm to (37.8, 17.0), turned to 0 degrees
Connections:
- removed net N$1: JP1.3
- removed net N$2: U$1.15
- removed net N$6: JP1.1
- new net PC2/ADC11: JP1.3, U$1.15
- net PC1/SCL/ADC10: now also JP1.1
Other:
- board text added: "PA7 PA6 PA5 PA4 PA3 PA2 PA1 PA0 PC2 PC1"
- board text added: "PC1 PC2 PA0 PA1 PA2 PA3 PA4 PA5 PA6 PA7"
- board text removed: "PA7 PA6 PA5 PA4 PA3 PA2 PA1 PA0 PXX PXX"
- board text removed: "PXX PXX PA0 PA1 PA2 PA3 PA4 PA5 PA6 PA7"
